Commit message: feat(sim): add two-way contact dynamics and scooper mass

File: ur_urdf/ur5_with_scoop.urdf (robot description, URDF)
Before this commit: robot ur5_with_scoop, 13 links, 12 joints
Links:
- link scoop_link: mass 0.5 -> 0.11

File: ur_urdf/ur5_with_scoop_v2.urdf (robot description, URDF)
Before this commit: robot ur5_with_scoop, 13 links, 12 joints
Links:
- link scoop_link: mass 0.5 -> 0.11

Commit message: Paths updated, mass updated

File: ur_urdf/ur5_with_scoop.urdf (robot description, URDF)
Before this commit: robot ur5_with_scoop, 13 links, 12 joints
Links:
- link base_link_inertia: geometry collision mesh filename=base.stl
- link forearm_link: geometry collision mesh filename=forearm.stl
- link scoop_link: geometry collision mesh filename=ur5_scoop.stl scale=0.001 0.001 0.001
- link shoulder_link: geometry collision mesh filename=shoulder.stl
- link upper_arm_link: geometry collision mesh filename=upperarm.stl
- link wrist_1_link: geometry collision mesh filename=wrist1.stl
- link wrist_2_link: geometry collision mesh filename=wrist2.stl
- link wrist_3_link: geometry collision mesh filename=wrist3.stl
